File: Autopilot_H743_V2.kicad_sch (KiCad schematic)
At the start: 226 parts, among them J2 XT30PW-M / 5V INPUT, J3 TYPE-C-31-M-12, J4 TF-01A / microSD, Q1 AO3401A, Q2 MMBT3906 PNP, Q3 MMBT2222A NPN, SW1 RESET, SW2 BOOT, U1 STM32H743VIT6, U10 BMI088, U11 MMC5983MA, U12 SPA06-003, U13 USBLC6-2SC6, U14 USBLC6-2SC6, U15 USBLC6-2SC6, U16 USBLC6-2SC6, U17 USBLC6-2SC6, U18 USBLC6-2SC6, U19 TPS2553DBVR, U2 AP63203WU-7, U20 USBLC6-2SC6, U21 SN74LV8T245PWR, U22 TMUX1574PWR, U23 TMUX1574PWR, U3 TPS2113APWR, U4 TPS7A2033PDBVR, U5 TUSB320LIRWBR, U6 TPS2553DBVR, U7 USBLC6-2SC6, U8 USBLC6-2SC6, U9 TPS7A2033PDBVR, Y1 8MHz

Commit message: Redraw v2 with the original MCU and boxed subsystems
Restore one original STM32H743 symbol with labeled signals and local bypass capacitors. Draw 22 rectangular subsystem blocks with labeled interfaces and short, explicit local wiring. Update the schematic preview and synchronize generated MCU no-connect net names in the PCB.

Validation: zero ERC violations; all 137 named v1 nets, 624 connected pins and 44 unused pins preserved after the approved connector-to-pad and XT30 mapping. Existing v2 BOM and connectivity are unchanged. Zero PCB schematic parity issues. PCB geometry is unchanged; placement/routing are unfinished and DRC has not passed (one clearance violation and 487 unconnected items).
Parts:
- removed unit 6 of U1
- removed unit 7 of U1
- removed unit 15 of U1
- removed unit 12 of U1
- removed unit 9 of U1
- removed unit 2 of U1
- removed unit 18 of U1
- removed unit 8 of U1
- removed unit 20 of U1
- removed unit 10 of U1
- removed unit 5 of U1
- removed unit 19 of U1
- removed unit 17 of U1
- removed unit 3 of U1
- removed unit 14 of U1
- removed unit 16 of U1
- removed unit 4 of U1
- removed unit 13 of U1
- removed unit 11 of U1
Connections:
- net ACTUATOR_OE_N: now also U1.57 (PD10)
- net ADC_BATT_I: now also U1.16 (PC1)
- net ADC_BATT_V: now also U1.15 (PC0)
- net BOOT0: now also U1.94 (BOOT0)
- net GND: now also U1.10 (VSS), U1.19 (VSSA), U1.26 (VSS), U1.49 (VSS), U1.74 (VSS), U1.99 (VSS)
- net HSE_IN: now also U1.12 (PH0)
- net HSE_OUT: now also U1.13 (PH1)
- net I2C1_SCL: now also U1.92 (PB6)
- net I2C1_SDA: now also U1.93 (PB7)
- net I2C2_SCL: now also U1.46 (PB10)
- net I2C2_SDA: now also U1.47 (PB11)
- net IMU_ACC_CS_N: now also U1.9 (PC15)
- net IMU_ACC_INT: now also U1.7 (PC13)
- net IMU_GYR_CS_N: now also U1.8 (PC14)
- net IMU_GYR_INT: now also U1.1 (PE2)
- net MAG_INT: now also U1.3 (PE4)
- net NRST: now also U1.14 (NRST)
- net OTG_FS_DM: now also U1.70 (PA11)
- net OTG_FS_DP: now also U1.71 (PA12)
- net OUT_BANK1_DSHOT: now also U1.58 (PD11)
- net OUT_BANK2_DSHOT: now also U1.84 (PD3)
- net PERIPH_FAULT_N: now also U1.4 (PE5)
- net PWM1_MCU: now also U1.22 (PA0)
- net PWM2_MCU: now also U1.23 (PA1)
- net PWM3_MCU: now also U1.24 (PA2)
- net PWM4_MCU: now also U1.25 (PA3)
- net PWM5_MCU: now also U1.59 (PD12)
- net PWM6_MCU: now also U1.60 (PD13)
- net PWM7_MCU: now also U1.61 (PD14)
- net PWM8_MCU: now also U1.62 (PD15)
- net SDMMC1_CK: now also U1.80 (PC12)
- net SDMMC1_CMD: now also U1.83 (PD2)
- net SDMMC1_D0: now also U1.65 (PC8)
- net SDMMC1_D1: now also U1.66 (PC9)
- net SDMMC1_D2: now also U1.78 (PC10)
- net SDMMC1_D3: now also U1.79 (PC11)
- net SD_DETECT_N: now also U1.95 (PB8)
- net SPI1_MISO: now also U1.30 (PA6)
- net SPI1_MOSI: now also U1.88 (PD7)
- net SPI1_SCK: now also U1.29 (PA5)
- net STATUS_LED: now also U1.2 (PE3)
- net SWCLK: now also U1.76 (PA14)
- net SWDIO: now also U1.72 (PA13)
- net UART7_RX: now also U1.37 (PE7)
- net UART7_TX: now also U1.38 (PE8)
- net UART8_RX: now also U1.97 (PE0)
- net UART8_TX: now also U1.98 (PE1)
- net USART1_RX: now also U1.69 (PA10)
- net USART1_TX: now also U1.68 (PA9)
- net USART2_RX: now also U1.87 (PD6)
- net USART2_TX: now also U1.86 (PD5)
- net USART3_RX: now also U1.56 (PD9)
- net USART3_TX: now also U1.55 (PD8)
- net USART6_RX: now also U1.64 (PC7)
- net USART6_TX: now also U1.63 (PC6)
- net USB_FAULT_N: now also U1.5 (PE6)
- net USB_PRESENT_N: now also U1.32 (PC4)
- net V3V3_CORE: now also U1.100 (VDD), U1.11 (VDD), U1.20 (VREF+), U1.21 (VDDA), U1.27 (VDD), U1.50 (VDD), U1.6 (VBAT), U1.75 (VDD)
- net VCAP_48: now also U1.48 (VCAP)
- net VCAP_73: now also U1.73 (VCAP)
Other:
- note added: "01 MCU / local bypass"
- note added: "02 Regulated 5V input / source selection"
- note added: "03 3.3V buck regulator"
- note added: "04 USB-C current detection / controller supply"
- note added: "05 Sensor supply / BMI088 IMU"
- note added: "06 MCU clock / reset / boot / debug"
- note added: "07 USB-C connector / data and CC protection"
- note added: "08 USB bench-power enable / current limit"
- note added: "09 Compass / barometer / I2C2 pullups"
- note added: "10 microSD / SDMMC"
- note added: "11 Peripheral 5V / USB-present detection"
- note added: "12 External I2C / battery-monitor inputs"
- note added: "13 UART7 / 3.3V UART"
- note added: "14 USART1 / 3.3V UART"
- note added: "15 USART2 / 3.3V UART"
- note added: "16 USART3 / 3.3V UART"
- note added: "17 UART8 / 3.3V UART"
- note added: "18 USART6 / 3.3V UART"
- note added: "19 Eight-channel 3.3V → 5V PWM buffer"
- note added: "20 Output bank 1 / PWM or bidirectional DShot"
- note added: "21 Output bank 2 / PWM or bidirectional DShot"
- note added: "22 Servo power pads / electrical notes"
- note added: "8MHz crystal: keep loop short. SWD 3V3 pad is a voltage reference. Hold BOOT, pulse RESET for ROM loader."
- note added: "Battery inputs: conditioned 0–3.3V only. 6S / 60A monitor remains external."
- note added: "C4 connects BST to SW. Keep input / switching loops short. Take feedback from the output capacitors; keep SW away from sensors. Bulk capacitors retain their v1 packages and ratings."
- note added: "CC_HIGH_CURRENT_N permits bench power when Type-C advertises 1.5A / 3A."
- note added: "DIR tied high: A→B. OE high disables buffer and both output selectors."
- note added: "Default-current USB hosts may not supply the complete board load."
- note added: "Keep barometer port clear. Place compass away from power-current loops."
- note added: "No CLK pullup. 33Ω series resistors at MCU; bypass at card socket."
- note added: "No IMU heater. Place bypass at supply pins; keep buck heat away."
- note added: "OUT 1"
- note added: "OUT 2"
- note added: "OUT 3"
- note added: "OUT 4"
- note added: "OUT 5"
- note added: "OUT 6"
- note added: "OUT 7"
- note added: "OUT 8"
- note added: "One physical STM32H743VIT6, original v1 symbol and pinout. C9–C16: 100nF per supply pin; place at the pin on PCB. NC crosses retain the intentionally unused v1 pins."
- note added: "SEL low = 5V PWM; high = direct 3.3V DShot. OE high = disabled."
- note added: "TX/RX names are from the autopilot. V5_PERIPH shared across ports."
- note added: "USB data: route as a 90Ω differential pair; minimize stubs. ESD parts at connector. R18 / R19 near MCU. USB-C and bench-power behavior are retained from v1."
- note added: "V5_PERIPH is main-powered only. ~0.5A shared by all ports. USB_PRESENT_N is active low."
- note added: "VCAP: 2.2uF each; no external load."
- note added: "VREF+ / pin 20"
- note added: "V_SERVO_BEC is isolated from V5_SYS; grounds are common. External BEC provides servo power. XT30 powers avionics at 5V. TP pads: 1.8mm copper, no paste; add wire strain relief. Signal names and pin assignments match v1. No heater fitted. PCB starter remains unplaced / unrouted; DRC is not passed."
- note added: "XT30: pin 2 +5V, pin 1 GND. Regulated 4.75–5.25V only."
- note added: "pin 100"
- note added: "pin 11"
- note added: "pin 21"
- note added: "pin 27"
- note added: "pin 50"
- note added: "pin 6"
- note added: "pin 75"
- note removed: "01 XT30 / input protection / source selection"
- note removed: "02 3.3V buck / local switching loop"
- note removed: "03 MCU power / bypass at each physical pin"
- note removed: "04 USB-C control supply / current advertisement"
- note removed: "05 USB bench-power switch / fault reporting"
- note removed: "06 USB-C / protection / MCU USB pins"
- note removed: "07 8MHz / reset / boot / SWD solder pads"
- note removed: "08 Sensor LDO / BMI088 / MCU SPI"
- note removed: "09 Compass / barometer / MCU I2C2"
- note removed: "10 microSD / MCU SDMMC / local bypass"
- note removed: "100nF per VDD / VDDA / VREF+ / VBAT pin. VCAP: no external load."
- note removed: "11 UART7 / 3.3V serial solder pads"
- note removed: "12 USART1 / 3.3V serial solder pads"
- note removed: "13 USART2 / 3.3V serial solder pads"
- note removed: "14 USART3 / 3.3V serial solder pads"
- note removed: "15 UART8 / 3.3V serial solder pads"
- note removed: "16 USART6 / 3.3V serial solder pads"
- note removed: "17 Peripheral power / USB present"
- note removed: "18 External I2C / battery monitor solder pads"
- note removed: "19 Eight outputs / 5V PWM or direct 3.3V bidirectional DShot"
- note removed: "20 Unused MCU pins / design notes"
- note removed: "33u03a9 series resistors; no CLK pullup. Qualify SD clock after PCB routing."
- note removed: "90u03a9 differential USB. Protection at connector. USB-C retained."
- note removed: "ADC pads accept conditioned 0u20133.3V signals only. 6S/60A monitor stays external."
- note removed: "C4 returns to SW, not GND. Keep U2u2013C7 hot loop short. Sense 3V3 at C5/C6; keep switching copper away from IMU. Retain 0805 output/bulk capacitors and 0603 VCAP parts. Small 100nF capacitors: 0402 / 16V X7R."
- note removed: "Keep barometer port clear. Compass away from power currents."
- note removed: "No heater fitted. Isolate from buck heat; calibrate sensor temperature drift."
- note removed: "REVISION TWO u2014 SINGLE SHEET U1 units are functional sections of ONE STM32H743, not separate chips. All original MCU pin assignments and signal net names are retained. Signal paths are wired locally between MCU units, protection, passives and solder pads. Identical power/net labels connect regions on this sheet. No JST-GH connectors or servo headers. XT30 supplies regulated 5V avionics only. S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"
- note removed: "SWD 3V3 pad is a voltage reference. BOOT held + RESET enters ROM loader."
- note removed: "Select LOW = 5V PWM, HIGH = 3.3V DShot. OE HIGH disables all outputs. V_SERVO_BEC is isolated from V5_SYS; common GND."
- note removed: "TX/RX labels are from the flight controller. Cross to peripheral RX/TX. V5_PERIPH: external-main power only, ~0.5A total across all ports. Pads are 1.8mm exposed copper; provide wire strain relief."
- note removed: "USB bench power requires Type-C 1.5A/3A advertisement. Ordinary default-current USB hosts are not a full-power source."
- note removed: "XT30: pin 2 = +5V, pin 1 = GND REGULATED 4.75u20135.25V ONLY; no raw battery."
- moved on the sheet: C1, C10, C11, C12, C13, C14, C15, C16, C17, C18, C19, C2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

Commit message: Shrink v2 solder pads and place peripherals with M3 mounting
Use underside 1.2 mm signal and 1.5 mm power/ground pads, a 40 mm placement target and 30.5 mm mounting centres. Correct XT30 sourcing to AMASS XT30PW-M30.G.Y / C431092. Preserve existing internal footprint arrangement and project constraints.

ERC and schematic parity pass. DRC has NOT passed: 487 unconnected items remain, with internal placement and all routing still pending. Add top/bottom peripheral placement preview with simplified connector bodies.
Parts:
- J2: LCSC C42039231 -> C431092; LCSC Part # C42039231 -> C431092; MPN XT30PW-M -> XT30PW-M30.G.Y
- TP1, TP12, TP13, TP16, TP17, TP20, TP21, TP24, TP25, TP28, TP29, TP32, TP33, TP36, TP37, TP38, TP4, TP40, TP41, TP43, TP44, TP46, TP47, TP49, TP5, TP50, TP52, TP53, TP55, TP56, TP58, TP59, TP8, TP9: footprint Autopilot_H743_V2:SolderPad_D1.8mm -> Autopilot_H743_V2:SolderPad_D1.5mm
- TP10, TP11, TP14, TP15, TP18, TP19, TP2, TP22, TP23, TP26, TP27, TP3, TP30, TP31, TP34, TP35, TP39, TP42, TP45, TP48, TP51, TP54, TP57, TP6, TP60, TP7: footprint Autopilot_H743_V2:SolderPad_D1.8mm -> Autopilot_H743_V2:SolderPad_D1.2mm
Other:
- note added: "V_SERVO_BEC is isolated from V5_SYS; grounds are common. External BEC provides servo power. XT30 powers avionics at 5V. TP pads: 1.2mm signal / 1.5mm power and GND, underside; no paste. Add wire strain relief. Signal names and pin assignments match v1. No heater fitted. PCB: peripherals placed; internals unplaced / unrouted. DRC is not passed."
- note removed: "V_SERVO_BEC is isolated from V5_SYS; grounds are common. External BEC provides servo power. XT30 powers avionics at 5V. TP pads: 1.8mm copper, no paste; add wire strain relief. Signal names and pin assignments match v1. No heater fitted. PCB starter remains unplaced / unrouted; DRC is not passed."

Commit message: Use solder-pad 5V input and shared servo supply; DRC not passed
Replace XT30 with ordinary 4 x 4 mm power pads. Feed servo power from V5_MAIN_IN before avionics protection, retaining USB-only logic power. Add C47 local decoupling and power routing notes/preset. ERC and schematic parity pass; board remains unrouted with 490 unconnected items and 282 parked-component DRC violations.
Parts:
- added C47: 47uF, Autopilot_H743_V2:Capacitor_SMD__C_1206_3216Metric, symbol Autopilot_H743_V2:C47uF
- J2: value XT30PW-M / 5V INPUT -> 5V BEC INPUT PADS; footprint Autopilot_H743_V2:AMASS_XT30PW-M_1x02_P2.50mm_Horizontal -> Autopilot_H743_V2:PowerInput_2Pad_4x4mm_P7mm; symbol Autopilot_H743_V2:XT30_J2 -> Autopilot_H743_V2:POWER_PADS_J2; LCSC C431092 -> (none); LCSC Part # C431092 -> (none); MPN XT30PW-M30.G.Y -> (none); Rating XT30PW-M / 5V INPUT -> Regulated 4.75-5.25 V; shared avionics and servo input; now left out of the parts list
- TP38, TP41, TP44, TP47, TP50, TP53, TP56, TP59: value V_SERVO_BEC -> V5_MAIN_IN; Rating V_SERVO_BEC -> V5_MAIN_IN
Connections:
- net V_SERVO_BEC is gone; now on net V5_MAIN_IN: TP38.1, TP41.1, TP44.1, TP47.1, TP50.1, TP53.1, TP56.1, TP59.1
- net GND: now also C47.2
- net V5_MAIN_IN: now also C47.1
Other:
- note added: "J2: pad 2 +5V, pad 1 GND. Regulated 4.75-5.25 V only. Servo feed branches BEFORE F1."
- note added: "V5_MAIN_IN feeds servos directly from J2; USB powers avionics only. Servo current bypasses F1, Q1 and U3; no onboard servo fuse or reverse protection. Route +5V and GND with broad copper; size both for combined stall/startup current. Return servo current toward J2, away from sensor circuitry; use parallel vias if needed. BEC / servo models TBD: current rating and wire size require final verificat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"
- note removed: "V_SERVO_BEC is isolated from V5_SYS; grounds are common. External BEC provides servo power. XT30 powers avionics at 5V. TP pads: 1.2mm signal / 1.5mm power and GND, underside; no paste. Add wire strain relief. Signal names and pin assignments match v1. No heater fitted. PCB: peripherals placed; internals unplaced / unrouted. DRC is not passed."
- note removed: "XT30: pin 2 +5V, pin 1 GND. Regulated 4.75–5.25V only."
Changed lines of the file:
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@@
 	(generator_version "9.0")
 	(paper "User" 1189 860)
-	(title_block
-		(title "H743 compact autopilot — revision two")
-		(date "2026-10-12")
-		(rev "2")
-		(company "Joseph Stewart")
-		(comment 1 "Regulated 5V XT30 input | USB-C | labeled subsystem interfaces | prototype")
-	)
+	(title_block (title "H743 compact autopilot — revision two") (date "2026-10-12") (rev "2") (company "Joseph Stewart") (comment 1 "Regulated 5V solder-pad input | USB-C | labeled subsystem interfaces | prototype"))
 	(rectangle
 		(start 706.12 622.3)
@@
 		)
 	)
-	(text "XT30: pin 2 +5V, pin 1 GND. Regulated 4.75–5.25V only."
-		(exclude_from_sim no)
-		(at 251.46 208.28 0)
-		(effects
-			(font
-				(size 0.95 0.95)
-			)
-			(justify left top)
-		)
-	)
+	(text "J2: pad 2 +5V, pad 1 GND. Regulated 4.75-5.25 V only. Servo feed branches BEFORE F1." (exclude_from_sim no) (at 251.46 208.28 0) (effects (font (size 0.95 0.95)) (justify left top)))
 	(text "VREF+ / pin 20"
 		(exclude_from_sim no)
@@
 		)
 	)
-	(text "V_SERVO_BEC is isolated from V5_SYS; grounds are common.\nExternal BEC provides servo power. XT30 powers avionics at 5V.\nTP pads: 1.2mm signal / 1.5mm power and GND, underside; no paste. Add wire strain relief.\nSignal names and pin assignments match v1. No heater fitted.\nPCB: peripherals placed; internals unplaced / unrouted. DRC is not passed."
-		(exclude_from_sim no)
-		(at 944.88 762 0)
-		(effects
-			(font
-				(size 0.98 0.98)
-			)
-			(justify left top)
-		)
-	)
+	(text "V5_MAIN_IN feeds servos directly from J2; USB powers avionics only.\nServo current bypasses F1, Q1 and U3; no onboard servo fuse or reverse protection.\nRoute +5V and GND with broad copper; size both for combined stall/startup current.\nReturn servo current toward J2, away from sensor circuitry; use parallel vias if needed.\nBEC / servo models TBD: current rating and wire size require final verification.\nC47 is local decoupling; allow for DC-bias loss. Check BEC sag and transients under load.\nTP pads: 1.2mm signal / 1.5mm power and GND, underside, no paste; strain-relieve wires.\nNo heater. Internals unplaced / unrouted. DRC is not passed." (exclude_from_sim no) (at 944.88 762 0) (effects (font (size 0.98 0.98)) (justify left top)))
 	(text "12  External I2C / battery-monitor inputs"
 		(exclude_from_sim no)
@@
 		)
 	)
-	(label "V_SERVO_BEC"
+	(label "V5_MAIN_IN"
 		(at 977.9 731.52 180)
 		(effects
@@
 		)
 	)
-	(label "V_SERVO_BEC"
+	(label "V5_MAIN_IN"
 		(at 1074.42 706.12 180)
 		(effects
@@
 		)
 	)
-	(label "V_SERVO_BEC"
+	(label "V5_MAIN_IN"
 		(at 977.9 655.32 180)
 		(effects
@@
 		)
 	)
-	(label "V_SERVO_BEC"
+	(label "V5_MAIN_IN"
 		(at 1074.42 680.72 180)
 		(effects
@@
 		)
 	)
-	(label "V_SERVO_BEC"
+	(label "V5_MAIN_IN"
 		(at 977.9 680.72 180)
 		(effects
@@
 		)
 	)
-	(label "V_SERVO_BEC"
+	(label "V5_MAIN_IN"
 		(at 977.9 706.12 180)
 		(effects
@@
 		)
 	)
-	(label "V_SERVO_BEC"
+	(label "V5_MAIN_IN"
 		(at 1074.42 731.52 180)
 		(effects
@@
 		)
 	)
-	(label "V_SERVO_BEC"
+	(label "V5_MAIN_IN"
 		(at 1074.42 655.32 180)
 		(effects
@@
 			)
 		)
-		(property "Value" "V_SERVO_BEC"
+		(property "Value" "V5_MAIN_IN"
 			(at 1089.66 732.79 0)
 			(effects
@@
 			)
 		)
-		(property "Rating" "V_SERVO_BEC"
+		(property "Rating" "V5_MAIN_IN"
 			(at 1082.04 731.52 0)
 			(effects
@@
 			)
 		)
-		(property "Value" "V_SERVO_BEC"
+		(property "Value" "V5_MAIN_IN"
 			(at 1089.66 707.39 0)
 			(effects
@@
 			)
 		)
-		(property "Rating" "V_SERVO_BEC"
+		(property "Rating" "V5_MAIN_IN"
 			(at 1082.04 706.12 0)
 			(effects
@@
 			)
 		)
-		(property "Value" "V_SERVO_BEC"
+		(property "Value" "V5_MAIN_IN"
 			(at 993.14 707.39 0)
 			(effects
@@
 			)
 		)
-		(property "Rating" "V_SERVO_BEC"
+		(property "Rating" "V5_MAIN_IN"
 			(at 985.52 706.12 0)
 			(effects
@@
 		)
 	)
-	(symbol
-		(lib_id "Autopilot_H743_V2:XT30_J2")
-		(at 269.24 86.36 0)
-		(unit 1)
-		(exclude_from_sim no)
-		(in_bom yes)
-		(on_board yes)
-		(dnp no)
-		(property "Reference" "J2"
-			(at 274.32 58.42 0)
-			(effects
-				(font
-					(size 1 1)
-				)
-			)
-		)
-		(property "Value" "XT30PW-M / 5V INPUT"
-			(at 274.32 62.23 0)
-			(effects
-				(font
-					(size 0.95 0.95)
-				)
-			)
-		)
-		(property "Footprint" "Autopilot_H743_V2:AMASS_XT30PW-M_1x02_P2.50mm_Horizontal"
-			(at 269.24 86.36 0)
-			(effects
-				(font
-					(size 1 1)
-				)
-				(hide yes)
-			)
-		)
-		(property "Datasheet" "https://datasheet.lcsc.com/datasheet/pdf/f40c503d729038bd14858056d73ccb74.pdf"
-			(at 269.24 86.36 0)
-			(effects
-				(font
-					(size 1 1)
-				)
-				(hide yes)
-			)
-		)
-		(property "Description" ""
-			(at 269.24 86.36 0)
-			(effects
-				(font
-					(size 1.27 1.27)
-				)
-			)
-		)
-		(property "LCSC" "C431092"
-			(at 269.24 86.36 0)
-			(effects
-				(font
-					(size 1 1)
-				)
-				(hide yes)
-			)
-		)
-		(property "LCSC Part #" "C431092"
-			(at 269.24 86.36 0)
-			(effects
-				(font
-					(size 1 1)
-				)
-				(hide yes)
-			)
-		)
-		(property "MPN" "XT30PW-M30.G.Y"
-			(at 269.24 86.36 0)
-			(effects
-				(font
-					(size 1 1)
-				)
-				(hide yes)
-			)
-		)
-		(property "Rating" "XT30PW-M / 5V INPUT"
-			(at 269.24 86.36 0)
-			(effects
-				(font
-					(size 1 1)
-				)
-				(hide yes)
-			)
-		)
-		(property "V1 Interface" ""
-			(at 269.24 86.36 0)
-			(effects
-				(font
-					(size 1 1)
-				)
-				(hide yes)
-			)
-		)
-		(pin "2"
-		)
-		(pin "1"
-		)
-		(instances
-			(project "Autopilot_H743_V2"
-				(path "/392c7d53-abcb-5d13-97f4-bb795b133b79"
-					(reference "J2")
-					(unit 1)
-				)
-			)
-		)
-	)
+	(symbol (lib_id "Autopilot_H743_V2:POWER_PADS_J2") (at 269.24 86.36 0) (unit 1) (exclude_from_sim no) (in_bom no) (on_board yes) (dnp no) (property "Reference" "J2" (at 274.32 58.42 0) (effects (font (size 1 1)))) (property "Value" "5V BEC INPUT PADS" (at 274.32 62.23 0) (effects (font (size 0.95 0.95)))) (property "Footprint" "Autopilot_H743_V2:PowerInput_2Pad_4x4mm_P7mm" (at 269.24 86.36 0) (effects (font (size 1 1)) (hide yes))) (property "Datasheet" "" (at 269.24 86.36 0) (effects (font (size 1 1)) (hide yes))) (property "Description" "Two ordinary top-side copper solder pads; hand solder wires; no paste or purchased connector" (at 269.24 86.36 0) (effects (font (size 1.27 1.27)) (hide yes))) (property "LCSC" "" (at 269.24 86.36 0) (effects (font (size 1 1)) (hide yes))) (property "LCSC Part #" "" (at 269.24 86.36 0) (effects (font (size 1 1)) (hide yes))) (property "MPN" "" (at 269.24 86.36 0) (effects (font (size 1 1)) (hide yes))) (property "Rating" "Regulated 4.75-5.25 V; shared avionics and servo input" (at 269.24 86.36 0) (effects (font (size 1 1)) (hide yes))) (property "V1 Interface" "" (at 269.24 86.36 0) (effects (font (size 1 1)) (hide yes))) (pin "2") (pin "1") (instances (project "Autopilot_H743_V2" (path "/392c7d53-abcb-5d13-97f4-bb795b133b79" (reference "J2") (unit 1)))))
 	(symbol
 		(lib_id "Autopilot_H743_V2:MCU")
@@
 			)
 		)
-		(property "Value" "V_SERVO_BEC"
+		(property "Value" "V5_MAIN_IN"
 			(at 993.14 732.79 0)
 			(effects
@@
 			)
 		)
-		(property "Rating" "V_SERVO_BEC"
+		(property "Rating" "V5_MAIN_IN"
 			(at 985.52 731.52 0)
 			(effects
@@
 			)
 		)
-		(property "Value" "V_SERVO_BEC"
+		(property "Value" "V5_MAIN_IN"
 			(at 993.14 656.59 0)
 			(effects
@@
 			)
 		)
-		(property "Rating" "V_SERVO_BEC"
+		(property "Rating" "V5_MAIN_IN"
 			(at 985.52 655.32 0)
 			(effects
@@
 			)
 		)
-		(property "Value" "V_SERVO_BEC"
+		(property "Value" "V5_MAIN_IN"
 			(at 993.14 681.99 0)
 			(effects
@@
 			)
 		)
-		(property "Rating" "V_SERVO_BEC"
+		(property "Rating" "V5_MAIN_IN"
 			(at 985.52 680.72 0)
 			(effects
@@
 			)
 		)
-		(property "Value" "V_SERVO_BEC"
+		(property "Value" "V5_MAIN_IN"
 			(at 1089.66 656.59 0)
 			(effects
@@
 			)
 		)
-		(property "Rating" "V_SERVO_BEC"
+		(property "Rating" "V5_MAIN_IN"
 			(at 1082.04 655.32 0)
 			(effects
@@
 			)
 		)
-		(property "Value" "V_SERVO_BEC"
+		(property "Value" "V5_MAIN_IN"
 			(at 1089.66 681.99 0)
 			(effects
@@
 			)
 		)
-		(property "Rating" "V_SERVO_BEC"
+		(property "Rating" "V5_MAIN_IN"
 			(at 1082.04 680.72 0)
 			(effects
@@
 	)
 	(embedded_fonts no)
+(symbol (lib_id "Autopilot_H743_V2:C47uF") (at 1120.1400 779.7800 0) (unit 1) (exclude_from_sim no) (in_bom yes) (on_board yes) (dnp no) (property "Reference" "C47" (at 1127.7600 777.2400 0) (effects (font (size 1 1)) (justify left))) (property "Value" "47uF" (at 1127.7600 781.0500 0) (effects (font (size 0.95 0.95)) (justify left))) (property "Footprint" "Autopilot_H743_V2:Capacitor_SMD__C_1206_3216Metric" (at 1120.1400 779.7800 0) (effects (font (size 1 1)) (hide yes))) (property "Datasheet" "https://www.lcsc.com/datasheet/C96123.pdf" (at 1120.1400 779.7800 0) (effects (font (size 1 1)) (hide yes))) (property "Description" "" (at 1120.1400 779.7800 0) (effects (font (size 1.27 1.27)))) (property "LCSC" "C96123" (at 1120.1400 779.7800 0) (effects (font (size 1 1)) (hide yes))) (property "LCSC Part #" "C96123" (at 1120.1400 779.7800 0) (effects (font (size 1 1)) (hide yes))) (property "MPN" "CL31A476MPHNNNE" (at 1120.1400 779.7800 0) (effects (font (size 1 1)) (hide yes))) (property "Rating" "47uF / 10V X5R; DC-bias derating applies" (at 1120.1400 779.7800 0) (effects (font (size 1 1)) (hide yes))) (property "V1 Interface" "" (at 1120.1400 779.7800 0) (effects (font (size 1 1)) (hide yes))) (pin "1") (pin "2") (instances (project "Autopilot_H743_V2" (path "/392c7d53-abcb-5d13-97f4-bb795b133b79" (reference "C47") (unit 1)))))
+(wire(pts(xy 1120.14 775.97)(xy 1120.14 768.35))(stroke(width 0)(type default)))
+(label "V5_MAIN_IN"(at 1120.14 768.35 0)(effects(font(size .95 .95))(justify left bottom)))
+(wire(pts(xy 1120.14 783.59)(xy 1120.14 791.21))(stroke(width 0)(type default)))
+(label "GND"(at 1120.14 791.21 0)(effects(font(size .95 .95))(justify left bottom)))
 )

Commit message: Expand v2 to 60mm with 50mm M3 mounting; DRC not passed
Redistribute underside peripheral pads at 3mm column pitch, 7mm UART row pitch and 5mm servo row pitch. Move power pads, USB-C and microSD to the new edges. Preserve the saved internal placements and project settings. ERC passes and all 180 nets are unchanged; internal placement and routing remain unfinished, with 490 unconnected items.
Changed lines of the file:
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@@
 		)
 	)
-	(text "V5_MAIN_IN feeds servos directly from J2; USB powers avionics only.\nServo current bypasses F1, Q1 and U3; no onboard servo fuse or reverse protection.\nRoute +5V and GND with broad copper; size both for combined stall/startup current.\nReturn servo current toward J2, away from sensor circuitry; use parallel vias if needed.\nBEC / servo models TBD: current rating and wire size require final verification.\nC47 is local decoupling; allow for DC-bias loss. Check BEC sag and transients under load.\nTP pads: 1.2mm signal / 1.5mm power and GND, underside, no paste; strain-relieve wires.\nNo heater. Internals unplaced / unrouted. DRC is not passed." (exclude_from_sim no) (at 944.88 762 0) (effects (font (size 0.98 0.98)) (justify left top)))
+	(text "V5_MAIN_IN feeds servos directly from J2; USB powers avionics only.\nServo current bypasses F1, Q1 and U3; no onboard servo fuse or reverse protection.\nRoute +5V and GND with broad copper; size both for combined stall/startup current.\nReturn servo current toward J2, away from sensor circuitry; use parallel vias if needed.\nBEC / servo models TBD: current rating and wire size require final verification.\nC47 is local decoupling; allow for DC-bias loss. Check BEC sag and transients under load.\nTP pads: 1.2mm signal / 1.5mm power and GND, underside, no paste; strain-relieve wires.\n60 x 60mm PCB; custom 50 x 50mm M3 mounting. No heater.\nInternals unplaced / unrouted. DRC is not passed." (exclude_from_sim no) (at 944.88 762 0) (effects (font (size 0.98 0.98)) (justify left top)))
 	(text "12  External I2C / battery-monitor inputs"
 		(exclude_from_sim no)
